Commit message: Updated URDF

File: controls/vis_gui/caster.urdf (robot description, URDF)
Before this commit: robot lram caster, 2 links, 1 joints
Links:
- link arm: geometry visual box size=.025 .025 .435
Joints:
- removed joint robot_arm
- added joint head_swivel: type continuous, parent base_link, child arm, origin xyz=0.0 0.125 0, axis 0 1 0
